File: build/4-tme-KiCad/4-tme-KiCad.kicad_sch (KiCad schematic)
At the start: 192 parts, among them J1 MIDI IN, J2 PITCH CV 1, J3 PITCH CV 2, J4 PITCH CV 3, J5 PITCH CV 4, SW1 RotaryEncoder, SW10 RotaryEncoder, SW11 RotaryEncoder, SW12 RotaryEncoder, SW13 RotaryEncoder, SW14 RotaryEncoder, SW15 RotaryEncoder, SW16 RotaryEncoder, SW17 RotaryEncoder, SW2 RotaryEncoder, SW3 RotaryEncoder, SW4 RotaryEncoder, SW5 RotaryEncoder, SW6 RotaryEncoder, SW7 RotaryEncoder, SW8 RotaryEncoder, SW9 RotaryEncoder, U1 CD74HC4067M, U2 CD74HC4067M, U3 6N137, U4 PCA9685, U5 MCP23017_SO, U6 CD74HC4067M, U7 MCP6004

Commit message: CV inputs
Parts:
- added C46, C47: 100nF_0603_25V, Capacitor_SMD:C_0201_0603Metric, symbol PCM_4ms_Capacitor:10nF_0603_25V
- added C48, C49, C50, C51: 10nF_0603_25V, Capacitor_SMD:C_0201_0603Metric, symbol PCM_4ms_Capacitor:10nF_0603_25V
- added D16, D17, D18, D19, D20, D21, D22, D23: BAT54S, Package_TO_SOT_SMD:SOT-23, symbol Diode:BAT54S
- added J6: PITCH CV 1, symbol Connector_Audio:AudioJack3
- added J7: PITCH CV 2, symbol Connector_Audio:AudioJack3
- added J8: PITCH CV 3, symbol Connector_Audio:AudioJack3
- added J9: PITCH CV 4, symbol Connector_Audio:AudioJack3
- added R100, R101, R102, R103: 100k, Resistor_SMD:R_0201_0603Metric, symbol Device:R
- added R104, R105, R106, R107: 33k, Resistor_SMD:R_0201_0603Metric, symbol Device:R
- added R108, R109, R110, R111: 1k, Resistor_SMD:R_0201_0603Metric, symbol Device:R
- added U8: MCP6004, Package_SO:SOIC-14_3.9x8.7mm_P1.27mm, symbol Amplifier_Operational:MCP6004
Connections:
- net A3V3: now also C46.1, C47.1, D16.2 (K), D17.2 (K), D18.2 (K), D19.2 (K), D20.2 (K), D21.2 (K), D22.2 (K), D23.2 (K), U8.4 (V+)
- net AGND: now also C46.2, C47.2, C48.2, C49.2, C50.2, C51.2, D16.1 (A), D17.1 (A), D18.1 (A), D19.1 (A), D20.1 (A), D21.1 (A), D22.1 (A), D23.1 (A), J6.R, J6.S, J7.R, J7.S, J8.R, J8.S, J9.R, J9.S, R104.2, R105.2, R106.2, R107.2, U8.11 (V-)
- net C30: no longer C36.1, R69.2
- net C31: no longer C37.1, R70.2
- net MENU_ENC_A: now also C36.1, R69.2
- net MENU_ENC_B: now also C37.1, R70.2
- net at R88.2, R92.1, U7.3 (+): now also D16.3 (COM)
- net at R90.2, R94.1, U7.10 (+): now also D20.3 (COM)
- net at R91.2, R95.1, U7.12 (+): now also D22.3 (COM)
- net at R89.2, R93.1, U7.5 (+): now also D18.3 (COM)
- net FILTER_CV_4: now reaches U6.19 (I12)
- net FILTER_CV_4: now also C51.1, R111.2
- net FILTER_CV_3: now reaches U6.20 (I11)
- net FILTER_CV_3: now also C50.1, R110.2
- net FILTER_CV_2: now reaches U6.21 (I10)
- net FILTER_CV_2: now also C49.1, R109.2
- net FILTER_CV_1: now reaches U6.22 (I9)
- net FILTER_CV_1: now also C48.1, R108.2
- new net: R109.1, U8.6 (-), U8.7
- new net: R108.1, U8.1, U8.2 (-)
- new net: J8.T, R102.1
- new net: D21.3 (COM), R102.2, R106.1, U8.10 (+)
- new net: R111.1, U8.13 (-), U8.14
- new net: J7.T, R101.1
- new net: J9.T, R103.1
- new net: D23.3 (COM), R103.2, R107.1, U8.12 (+)
- new net: J6.T, R100.1
- new net: R110.1, U8.8, U8.9 (-)
- new net: D17.3 (COM), R100.2, R104.1, U8.3 (+)
- new net: D19.3 (COM), R101.2, R105.1, U8.5 (+)
Other:
- note added: "FILTER CV"
- note added: "PITCH CV"
- moved on the sheet: C1, C2, C35, C42, C43, C44, C45, J2, J3, J4, J5, R88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
